Commit message: updated control

File: urdf/micromouse_robot.xacro (robot description, xacro)
@@ -45,44 +45,4 @@
   <xacro:wheel_y name="link_back_wheel" h="0.01" r="0.015" m="0.2" />
   <xacro:joint_wheel_y name="joint_back_wheel" parent="link_chassis" child="link_back_wheel" origin_xyz="0 -0.041 0" />
-  <transmission name="left_wheel_trans">
-     <type>transmission_interface/SimpleTransmission</type>
-     <actuator name="left_wheel_motor">
-       <hardwareInterface>VelocityJointInterface</hardwareInterface>
-       <mechanicalReduction>7</mechanicalReduction>
-     </actuator>
-     <joint name="joint_left_wheel">
-       <hardwareInterface>VelocityJointInterface</hardwareInterface>
-     </joint>
-  </transmission>
-  <transmission name="right_wheel_trans">
-     <type>transmission_interface/SimpleTransmission</type>
-     <actuator name="right_wheel_motor">
-       <hardwareInterface>VelocityJointInterface</hardwareInterface>
-       <mechanicalReduction>7</mechanicalReduction>
-     </actuator>
-     <joint name="joint_right_wheel">
-       <hardwareInterface>VelocityJointInterface</hardwareInterface>
-     </joint>
-  </transmission>
-  <transmission name="front_wheel_trans">
-     <type>transmission_interface/SimpleTransmission</type>
-     <actuator name="front_wheel_motor">
-       <hardwareInterface>VelocityJointInterface</hardwareInterface>
-       <mechanicalReduction>7</mechanicalReduction>
-     </actuator>
-     <joint name="joint_front_wheel">
-       <hardwareInterface>VelocityJointInterface</hardwareInterface>
-     </joint>
-  </transmission>
-  <transmission name="back_wheel_trans">
-     <type>transmission_interface/SimpleTransmission</type>
-     <actuator name="back_wheel_motor">
-       <hardwareInterface>VelocityJointInterface</hardwareInterface>
-       <mechanicalReduction>7</mechanicalReduction>
-     </actuator>
-     <joint name="joint_back_wheel">
-       <hardwareInterface>VelocityJointInterface</hardwareInterface>
-     </joint>
-  </transmission>
   <gazebo>
     <plugin filename="libgazebo_ros_diff_drive.so" name="differential_drive_controller">
@@ -91,7 +51,7 @@
       <leftJoint>joint_left_wheel</leftJoint>
       <rightJoint>joint_right_wheel</rightJoint>
-      <wheelSeparation>0.4</wheelSeparation>
-      <wheelDiameter>0.2</wheelDiameter>
-      <torque>0.1</torque>
+      <wheelSeparation>0.082</wheelSeparation>
+      <wheelDiameter>0.03</wheelDiameter>
+      <torque>10</torque>
       <commandTopic>cmd_vel_y</commandTopic>
       <odometryTopic>odom</odometryTopic>
@@ -106,7 +66,7 @@
       <leftJoint>joint_front_wheel</leftJoint>
       <rightJoint>joint_back_wheel</rightJoint>
-      <wheelSeparation>0.4</wheelSeparation>
-      <wheelDiameter>0.2</wheelDiameter>
-      <torque>0.1</torque>
+      <wheelSeparation>0.082</wheelSeparation>
+      <wheelDiameter>0.03</wheelDiameter>
+      <torque>10</torque>
       <commandTopic>cmd_vel_x</commandTopic>
       <odometryTopic>odom</odometryTopic>
@@ -159,5 +119,5 @@
         <range>
           <min>0.04</min>
-          <max>10.0</max>
+          <max>3.5</max>
           <resolution>0.01</resolution>
         </range>
